File: kicad/Euro2040.kicad_sch (KiCad schematic)
At the start: 39 parts

Commit message: save
Parts:
- removed J?: Conn_01x03_Female, symbol Connector:Conn_01x03_Female
- added C13: 2U2, Capacitor_SMD:C_0402_1005Metric, symbol Device:C
- added C19, C3: 10u, Capacitor_SMD:C_0805_2012Metric, symbol Device:C_Polarized
- added C20, C21, C22, C23: 100n, Capacitor_SMD:C_0402_1005Metric, symbol Device:C
- added D3, D4, D5: DIODE, Diode_SMD:D_0805_2012Metric, symbol Simulation_SPICE:DIODE
- added J3: Conn_02x05_Odd_Even, Eurorack:Eurorack Power Header Unlabeled, symbol Connector_Generic:Conn_02x05_Odd_Even
- added J5: Conn_01x10_Male, Connector_PinHeader_2.54mm:PinHeader_1x22_P2.54mm_Horizontal, symbol Connector:Conn_01x22_Male
- added R16, R17, R22, R23, R24, R25, R5, R6: 39K, Resistor_SMD:R_0402_1005Metric, symbol Device:R
- added R18, R19, R20, R21, R26, R27, R28, R29: 100K, Resistor_SMD:R_0402_1005Metric, symbol Device:R
- added U4: L7805, Package_TO_SOT_SMD:SOT-89-3, symbol Regulator_Linear:L7805
- added U5, U6: TL074, Package_SO:SOIC-14_3.9x8.7mm_P1.27mm, symbol Amplifier_Operational:TL074
- added U7: LM4040DBZ-3, Package_TO_SOT_SMD:SOT-23, symbol Reference_Voltage:LM4040DBZ-3
- C1, C10, C11, C12, C14, C15, C16, C17, C18, C2, C4, C5, C6, C7, C8, C9: renamed from C?; footprint (none) -> Capacitor_SMD:C_0402_1005Metric
- D1: renamed from D?; footprint (none) -> Diode_SMD:D_0805_2012Metric
- D2: renamed from D?; footprint (none) -> LED_SMD:LED_0402_1005Metric
- J1: renamed from J?; footprint (none) -> Connector_USB:USB_Micro-B_Amphenol_10103594-0001LF_Horizontal
- L1: renamed from L?; footprint (none) -> Inductor_SMD:L_0402_1005Metric
- R1, R10, R11, R12, R13, R14, R15, R2, R3, R4, R7, R8, R9: renamed from R?; footprint (none) -> Resistor_SMD:R_0402_1005Metric
- SW1: renamed from SW?; footprint (none) -> Button_Switch_SMD:SW_SPST_PTS810
- U1: renamed from U?; footprint RP2040_minimal:RP2040-QFN-56 -> rp2040:QFN40P700X700X90-57N
- U2: renamed from U?; footprint 10-WFDFN-EP_RIT -> RT6150B-33GQW:RT6150B-33GQW
- U3: renamed from U?; footprint W25Q16JVUXIQ_WIN -> w25q16jvuxiq:W25Q16JVUXIQ
- X1: renamed from Y?; footprint (none) -> Crystal:Crystal_SMD_3225-4Pin_3.2x2.5mm
Connections:
- net 3V3: now also J5.1 (Pin_1)
- net Earth: now also C13.2, C19.2, C20.2, C21.1, C22.2, C23.1, C3.1, J3.3 (Pin_3), J3.4 (Pin_4), J3.5 (Pin_5), J3.6 (Pin_6), J3.7 (Pin_7), J3.8 (Pin_8), J5.22 (Pin_22), J5.6 (Pin_6), R16.2, R17.2, R22.2, R23.2, R24.2, R25.2, R5.2, R6.2, U4.2 (GND), U7.2 (A)
- net GPIO_0: now also J5.7 (Pin_7), R18.2, U5.1; no longer U1.2 (GPIO0)
- net GPIO_1: now also J5.8 (Pin_8), R19.2, U5.7; no longer U1.3 (GPIO1)
- net GPIO_10: now also J5.17 (Pin_17)
- net GPIO_11: now also J5.18 (Pin_18)
- net GPIO_2: now also J5.9 (Pin_9), R20.2, U5.8; no longer U1.4 (GPIO2)
- net GPIO_26_ADC0: now also J5.2 (Pin_2), J5.5 (Pin_5)
- net GPIO_27_ADC0: now also J5.3 (Pin_3)
- net GPIO_3: now also J5.10 (Pin_10), R21.2, U5.14; no longer U1.5 (GPIO3)
- net GPIO_4: now also J5.11 (Pin_11), R26.2, U6.1; no longer U1.6 (GPIO4)
- net GPIO_5: now also J5.12 (Pin_12), R27.2, U6.7; no longer U1.7 (GPIO5)
- net GPIO_6: now also J5.13 (Pin_13), R28.2, U6.8; no longer U1.8 (GPIO6)
- net GPIO_7: now also J5.14 (Pin_14), R29.2, U6.14; no longer U1.9 (GPIO7)
- net GPIO_8: now also J5.15 (Pin_15)
- net GPIO_9: now also J5.16 (Pin_16)
- net VSYS: now also D5.2 (K)
- net at R9.2, U1.43 (ADC_AVDD): now also C13.1
- net ADC_VREF: no longer names the net of R7.2, R9.1
- net ADC_VREF: now also U7.1 (K)
- net GPIO_28\ADC0 renamed GPIO_28_ADC0
- net GPIO_28_ADC0: now also J5.4 (Pin_4)
- new net: R24.1, R28.1, U6.9 (-)
- new net: R17.1, R21.1, U5.13 (-)
- new net: D3.1 (A), J3.1 (Pin_1), J3.2 (Pin_2)
- new net: R16.1, R20.1, U5.9 (-)
- new net: R19.1, R6.1, U5.6 (-)
- new net: R22.1, R26.1, U6.2 (-)
- new net: R25.1, R29.1, U6.13 (-)
- new net: D4.2 (K), J3.10 (Pin_10), J3.9 (Pin_9)
- new net: R18.1, R5.1, U5.2 (-)
- new net: R23.1, R27.1, U6.6 (-)
- new net +12V: C19.1, C20.1, C22.1, D3.2 (K), J5.20 (Pin_20), U4.1 (IN), U5.4 (V+), U6.4 (V+)
- new net -12V: C21.2, C23.2, C3.2, D4.1 (A), J5.21 (Pin_21), U5.11 (V-), U6.11 (V-)
- new net GPIO_0X: U1.2 (GPIO0), U5.3 (+)
- new net GPIO_1X: U1.3 (GPIO1), U5.5 (+)
- new net GPIO_2X: U1.4 (GPIO2), U5.10 (+)
- new net GPIO_3X: U1.5 (GPIO3), U5.12 (+)
- new net GPIO_4X: U1.6 (GPIO4), U6.3 (+)
- new net GPIO_5X: U1.7 (GPIO5), U6.5 (+)
- new net GPIO_6X: U1.8 (GPIO6), U6.10 (+)
- new net GPIO_7X: U1.9 (GPIO7), U6.12 (+)
- new net V_7805: D5.1 (A), J5.19 (Pin_19), U4.3 (OUT)
Other:
- note added: "0 SCL"
- note added: "0 SDA"
- note added: "1 SCL"
- note added: "1 SDA"
- note added: "10V"
- moved on the sheet: C16, C17, R14, R15, R7, R9, X1

Commit message: more pins, output RC filter, pcb layout
Parts:
- removed C22, C23: 100n, Capacitor_SMD:C_0402_1005Metric, symbol Device:C
- added C24, C25, C26, C27, C28, C29, C30, C31: 100n, Capacitor_SMD:C_0402_1005Metric, symbol Device:C
- added R30, R31, R32, R33, R34, R35, R36, R37: 1K, Resistor_SMD:R_0402_1005Metric, symbol Device:R
- J5: footprint Connector_PinHeader_2.54mm:PinHeader_1x22_P2.54mm_Horizontal -> Connector_PinHeader_2.00mm:PinHeader_1x28_P2.00mm_Horizontal; symbol Connector:Conn_01x22_Male -> Connector:Conn_01x28_Male
Connections:
- net +12V: now also J5.26 (Pin_26); no longer J5.20 (Pin_20)
- net -12V: now also J5.27 (Pin_27); no longer J5.21 (Pin_21)
- net 3V3: now also J5.24 (Pin_24); no longer J5.1 (Pin_1)
- net Earth: now also J5.21 (Pin_21), J5.28 (Pin_28), C24.2, C25.2, C26.2, C27.2, C28.2, C29.2, C30.2, C31.2; no longer J5.22 (Pin_22), J5.6 (Pin_6)
- net GPIO_0: now also J5.5 (Pin_5); no longer J5.7 (Pin_7)
- net GPIO_0X: now also R30.2; no longer U5.3 (+)
- net GPIO_1: now also J5.6 (Pin_6); no longer J5.8 (Pin_8)
- net GPIO_10: now also J5.15 (Pin_15); no longer J5.17 (Pin_17)
- net GPIO_11: now also J5.16 (Pin_16); no longer J5.18 (Pin_18)
- net GPIO_12: now also J5.17 (Pin_17)
- net GPIO_13: now also J5.18 (Pin_18)
- net GPIO_14: now also J5.19 (Pin_19)
- net GPIO_15: now also J5.20 (Pin_20)
- net GPIO_1X: now also R31.2; no longer U5.5 (+)
- net GPIO_2: now also J5.7 (Pin_7); no longer J5.9 (Pin_9)
- net GPIO_26_ADC0: now also J5.1 (Pin_1), J5.4 (Pin_4); no longer J5.2 (Pin_2), J5.5 (Pin_5)
- net GPIO_27_ADC0: now also J5.2 (Pin_2); no longer J5.3 (Pin_3)
- net GPIO_28_ADC0: now also J5.3 (Pin_3); no longer J5.4 (Pin_4)
- net GPIO_2X: now also R32.2; no longer U5.10 (+)
- net GPIO_3: now also J5.8 (Pin_8); no longer J5.10 (Pin_10)
- net GPIO_3X: now also R33.2; no longer U5.12 (+)
- net GPIO_4: now also J5.9 (Pin_9); no longer J5.11 (Pin_11)
- net GPIO_4X: now also R34.2; no longer U6.3 (+)
- net GPIO_5: now also J5.10 (Pin_10); no longer J5.12 (Pin_12)
- net GPIO_5X: now also R35.2; no longer U6.5 (+)
- net GPIO_6: now also J5.11 (Pin_11); no longer J5.13 (Pin_13)
- net GPIO_6X: now also R36.2; no longer U6.10 (+)
- net GPIO_7: now also J5.12 (Pin_12); no longer J5.14 (Pin_14)
- net GPIO_7X: now also R37.2; no longer U6.12 (+)
- net GPIO_8: now also J5.13 (Pin_13); no longer J5.15 (Pin_15)
- net GPIO_9: now also J5.14 (Pin_14); no longer J5.16 (Pin_16)
- net USB_D+: now also J5.22 (Pin_22)
- net USB_D-: now also J5.23 (Pin_23)
- net V_7805: now also J5.25 (Pin_25); no longer J5.19 (Pin_19)
- new net: C30.1, R36.1, U6.10 (+)
- new net: C26.1, R32.1, U5.10 (+)
- new net: C27.1, R33.1, U5.12 (+)
- new net: C28.1, R34.1, U6.3 (+)
- new net: C24.1, R30.1, U5.3 (+)
- new net: C31.1, R37.1, U6.12 (+)
- new net: C29.1, R35.1, U6.5 (+)
- new net: C25.1, R31.1, U5.5 (+)
Other:
- note added: "I2C0 SCL"
- note added: "I2C0 SDA"
- note added: "I2C1 SCL"
- note added: "I2C1 SDA"
- note added: "SPI1 CSn"
- note added: "SPI1 RX"
- note added: "SPI1 SCK"
- note added: "SPI1 TX"
- note added: "UART0 RX"
- note added: "UART0 TX"
- note removed: "0 SCL"
- note removed: "0 SDA"
- note removed: "1 SCL"
- note removed: "1 SDA"
- moved on the sheet: C16, C17, C20, C21, C3, D2, R14, R15, R16, R17, R18, R19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
